Commit message: Rename to robo and edited amcl configs

File: 03_where_am_i/src/robo/urdf/my_robot.xacro (robot description, xacro)
@@ -1,5 +1,5 @@
 <?xml version='1.0'?>
-<robot name="my_robot" xmlns:xacro="http://www.ros.org/wiki/xacro">
-  <xacro:include filename="$(find my_robot)/urdf/my_robot.gazebo" />
+<robot name="robo" xmlns:xacro="http://www.ros.org/wiki/xacro">
+  <xacro:include filename="$(find robo)/urdf/robo.gazebo" />
   <link name="robot_footprint"></link>
   <joint name="robot_footprint_joint" type="fixed">
@@ -178,5 +178,5 @@
       <origin xyz="0 0 0" rpy="0 0 0"/>
       <geometry>
-        <mesh filename="package://my_robot/meshes/hokuyo.dae"/>
+        <mesh filename="package://robo/meshes/hokuyo.dae"/>
       </geometry>
     </visual>
