Commit message: updated camera link

File: 04_map_my_world/src/robo/urdf/robo.xacro (robot description, xacro)
@@ -161,5 +161,5 @@
   <joint name="camera_optical_joint" type="fixed">
     <origin xyz="0 0 0" rpy="-1.5707 0 -1.5707"/>
-    <parent link="camera_link"/>
+    <parent link="camera"/>
     <child link="camera_link_optical"/>
   </joint>
