Commit message: Use robo from 03

File: 05_home_service_robot/src/robo/urdf/robo.xacro (robot description, xacro)
@@ -1,5 +1,5 @@
 <?xml version='1.0'?>
-<robot name="homerobo" xmlns:xacro="http://www.ros.org/wiki/xacro">
-  <xacro:include filename="$(find homerobo)/urdf/homerobo.gazebo" />
+<robot name="robo" xmlns:xacro="http://www.ros.org/wiki/xacro">
+  <xacro:include filename="$(find robo)/urdf/robo.gazebo" />
   <link name="robot_footprint"></link>
   <joint name="robot_footprint_joint" type="fixed">
@@ -178,5 +178,5 @@
       <origin xyz="0 0 0" rpy="0 0 0"/>
       <geometry>
-        <mesh filename="package://homerobo/meshes/hokuyo.dae"/>
+        <mesh filename="package://robo/meshes/hokuyo.dae"/>
       </geometry>
     </visual>
